Commit message: More accurate coordinate systems
Correct orientations/lengths
Include search camera

File: src/ros/samplereturn/urdf/robot.xacro (robot description, xacro)
@@ -23,36 +23,15 @@
         <color rgba="0.1 0.8 0.2 1.0"/>
     </material>
-    <!-- the big triangle -->
-    <link name="base_link">
-        <inertial>
-            <origin xyz="0.75 0.5 0.05" />
-            <mass value="1.0" />
-            <inertia  ixx="0.140" ixy="0.0"  ixz="0.0"  iyy="0.105"  iyz="0.0" izz="0.246" />
-        </inertial>
-        <visual>
-            <origin xyz="0 0 0"/>
-            <geometry>
-                <mesh filename="package://samplereturn/Media/models/triangle.mesh.xml" />
-            </geometry>
-            <material name="plate"/>
-        </visual>
-        <collision>
-            <origin xyz="0 0 0"/>
-            <geometry>
-                <mesh filename="package://samplereturn/Media/models/triangle.mesh.xml" />
-            </geometry>
-        </collision>
-    </link>
     <xacro:macro name="wheel_module" params="name position">
         <joint name="${name}_suspension_joint" type="revolute">
             <axis xyz="0 0 1"/>
             <limit upper="1.57" lower="-1.57" effort="100" velocity="3.14"/>
-            <parent link="base_link"/>
+            <parent link="body_triangle"/>
             <child link="${name}_suspension"/>
-            <origin xyz="${position}"/>
+            <origin xyz="${position}" rpy="0 0 1.57"/>
         </joint>
         <link name="${name}_suspension">
             <visual>
-                <origin xyz="0 0 ${-suspension_height/2}"/>
+                <origin xyz="0 0 ${-suspension_height/2}" rpy="0 0 -1.57"/>
                 <geometry>
                     <cylinder length="${suspension_height}" radius="0.075"/>
@@ -166,4 +145,21 @@
         <!-- END RIGHT CAMERA -->
     </xacro:macro>
+    <link name="base_link">
+    </link>
+    <joint name="base_joint" type="fixed">
+        <parent link="base_link"/>
+        <child link="body_triangle"/>
+        <origin xyz="1.5 0 0" rpy="0 0 0.0"/>
+    </joint>
+    <!-- the big triangle -->
+    <link name="body_triangle">
+        <visual>
+            <origin xyz="0.0 -0.75 0" rpy="0 0 1.57"/>
+            <geometry>
+                <mesh filename="package://samplereturn/Media/models/triangle.mesh.xml" />
+            </geometry>
+            <material name="plate"/>
+        </visual>
+    </link>
     <!-- define suspension properties -->
     <xacro:property name="wheel_diameter" value="0.33"/>
@@ -172,12 +168,12 @@
     <xacro:property name="suspension_height" value="0.15"/>
     <!-- instantiate 3 modules -->
-    <xacro:wheel_module name="rear" position="0.75 1.30 0"/>
-    <xacro:wheel_module name="right_front" position="0.170 0.105 0"/>
-    <xacro:wheel_module name="left_front" position="1.330 0.105 0"/>
+    <xacro:wheel_module name="stern" position="-1.3 0 0"/>
+    <xacro:wheel_module name="port" position="0.0 0.5625 0"/>
+    <xacro:wheel_module name="starboard" position="0.0 -0.5625 0"/>
     <!-- instantiate navigation pair -->
     <xacro:stereo_pair name="navigation" baseline="0.30" />
     <!-- attach navigation pair -->
     <joint name="navigation_stereo_pair_joint" type="fixed">
-        <parent link="base_link"/>
+        <parent link="body_triangle"/>
         <child link="navigation_baseline_bar"/>
         <!-- macro defines camera with lenses facing along +z -->
@@ -189,5 +185,31 @@
         -->
         <!-- so camera should be at 1.4 - deck -->
-        <origin xyz="0.75 0.5 0.900" rpy="1.8588 0 0"/>
+        <origin xyz="0.015 0.0 0.990" rpy="1.745 0 1.57"/>
+    </joint>
+    <link name="search_camera_body">
+        <visual>
+            <geometry>
+                <box size="0.10 0.08 0.05"/>
+            </geometry>
+            <material name="sensor"/>
+        </visual>
+    </link>
+    <link name="search_camera_lens">
+        <visual>
+            <geometry>
+                <cylinder length="0.10" radius="0.035"/>
+            </geometry>
+            <material name="lens"/>
+        </visual>
+    </link>
+    <joint name="search_lens_joint" type="fixed">
+        <parent link="search_camera_body"/>
+        <child link="search_camera_lens"/>
+        <origin xyz="0.0 0.0 0.025" rpy="0 0 0"/>
+    </joint>
+    <joint name="search_camera_joint" type="fixed">
+        <parent link="body_triangle"/>
+        <child link="search_camera_body"/>
+        <origin xyz="0.10 0.0 1.0" rpy="1.65 0 1.57"/>
     </joint>
     <!-- carousel -->
@@ -195,5 +217,5 @@
         <visual>
             <geometry>
-                <cylinder length="0.250" radius="0.6"/>
+                <cylinder length="0.216" radius="0.406"/>
             </geometry>
             <material name="carousel"/>
@@ -201,8 +223,8 @@
     </link>
     <joint name="carousel_joint" type="continuous">
-        <parent link="base_link"/>
+        <parent link="body_triangle"/>
         <child link="carousel"/>
         <axis xyz="0 0 1"/>
-        <origin xyz="0.75 0.5 -0.125"/>
+        <origin xyz="-0.239 0.0 -0.121"/>
     </joint>
 </robot>

Commit message: Add manipulator camera
to launch and urdf

File: src/ros/samplereturn/urdf/robot.xacro (robot description, xacro)
@@ -85,5 +85,5 @@
         </link>
         <!-- BEGIN LEFT CAMERA -->
-        <joint name="${name_left_camera_joint" type="fixed">
+        <joint name="${name}_left_camera_joint" type="fixed">
             <parent link="${name}_baseline_bar"/>
             <child link="${name}_left_camera"/>
@@ -187,4 +187,20 @@
         <origin xyz="0.015 0.0 0.990" rpy="1.745 0 1.57"/>
     </joint>
+    <!-- instantiate manipulator pair -->
+    <xacro:stereo_pair name="manipulator" baseline="0.30" />
+    <!-- attach navigation pair -->
+    <joint name="manipulator_stereo_pair_joint" type="fixed">
+        <parent link="body_triangle"/>
+        <child link="manipulator_baseline_bar"/>
+        <!-- macro defines camera with lenses facing along +z -->
+        <!-- rpy is pi/2 + 16.5 degree down tilt -->
+        <!-- height of bottom of deck (origin) is -->
+        <!-- suspension_height + yoke_height - yoke_offset + wheel_radius -->
+        <!--
+        suspension_height+wheel_diameter*1.25/2-wheel_diameter*0.125/2+wheel_diameter/2
+        -->
+        <!-- so camera should be at 1.4 - deck -->
+        <origin xyz="-0.20 0.0 0.040" rpy="1.745 0 1.57"/>
+    </joint>
     <link name="search_camera_body">
         <visual>

Commit message: Fixed camera frames to match ROS convention and tilt angle

File: src/ros/samplereturn/urdf/robot.xacro (robot description, xacro)
@@ -88,5 +88,5 @@
             <parent link="${name}_baseline_bar"/>
             <child link="${name}_left_camera"/>
-            <origin xyz="${baseline/2} 0 0"/>
+            <origin xyz="${-baseline/2} 0 0"/>
         </joint>
         <link name="${name}_left_camera">
@@ -120,5 +120,5 @@
             <parent link="${name}_baseline_bar"/>
             <child link="${name}_right_camera"/>
-            <origin xyz="${-baseline/2} 0 0"/>
+            <origin xyz="${baseline/2} 0 0"/>
         </joint>
         <link name="${name}_right_camera">
@@ -185,5 +185,5 @@
         -->
         <!-- so camera should be at 1.4 - deck -->
-        <origin xyz="0.015 0.0 0.990" rpy="1.745 0 1.57"/>
+        <origin xyz="0.015 0.0 0.990" rpy="-2.00 0 -1.57"/>
     </joint>
     <!-- instantiate manipulator pair -->
@@ -201,5 +201,5 @@
         -->
         <!-- so camera should be at 1.4 - deck -->
-        <origin xyz="-0.20 0.0 0.040" rpy="1.745 0 1.57"/>
+        <origin xyz="-0.20 0.0 0.040" rpy="-2.80 0 -1.57"/>
     </joint>
     <link name="search_camera_body">
@@ -227,5 +227,5 @@
         <parent link="body_triangle"/>
         <child link="search_camera_body"/>
-        <origin xyz="0.10 0.0 1.0" rpy="1.65 0 1.57"/>
+        <origin xyz="0.10 0.0 1.0" rpy="-1.77 0 -1.57"/>
     </joint>
     <!-- carousel -->

Commit message: Change joint name to match joint_state report

File: src/ros/samplereturn/urdf/robot.xacro (robot description, xacro)
@@ -24,5 +24,5 @@
     </material>
     <xacro:macro name="wheel_module" params="name position">
-        <joint name="${name}_suspension_joint" type="revolute">
+        <joint name="${name}_steering_joint" type="revolute">
             <axis xyz="0 0 1"/>
             <limit upper="1.57" lower="-1.57" effort="100" velocity="3.14"/>

Commit message: Now the wheels sit on the ground

File: src/ros/samplereturn/urdf/robot.xacro (robot description, xacro)
@@ -3,5 +3,5 @@
 <robot
     xmlns:xacro="http://playerstage.sourceforge.net/gazebo/xmlschema/#interface"
-    name="awesome_robot">
+    name="">
     <enableGravity>false</enableGravity>
     <material name="plate">
@@ -33,7 +33,7 @@
         <link name="${name}_suspension">
             <visual>
-                <origin xyz="0 0 ${-suspension_height/2}" rpy="0 0 -1.57"/>
-                <geometry>
-                    <cylinder length="${suspension_height}" radius="0.075"/>
+                <origin xyz="0 0 ${-suspension_length/2}" rpy="0 0 -1.57"/>
+                <geometry>
+                    <cylinder length="${suspension_length}" radius="0.06"/>
                 </geometry>
                 <material name="suspension"/>
@@ -45,12 +45,11 @@
             <!-- z puts yoke at bottom of suspension since last number is
             yoke_height/2 -->
-            <origin xyz="0 0 ${-suspension_height-wheel_diameter*1.25/4}"/>
+            <origin xyz="0 0 ${-suspension_length}"/>
         </joint>
         <link name="${name}_yoke">
             <visual>
-                <geometry>
-                    <!-- 2.25 and 1.25 are aribtrary factors to make things look nice -->
-                    <!-- be sure to check _yoke_joint and _axle if you change z -->
-                    <box size="${wheel_width*2.25} ${yoke_thickness} ${wheel_diameter*1.25/2}"/>
+                <origin xyz="0 0 ${-yoke_height/2}" rpy="0 0 0"/>
+                <geometry>
+                    <box size="0.18 0.15 ${yoke_height}"/>
                 </geometry>
                 <material name="suspension"/>
@@ -63,5 +62,5 @@
             <child link="${name}_wheel"/>
             <!-- 1.25 must match factor in yoke, 0.125 is (1.25-1)/2 -->
-            <origin xyz="0 0 ${-wheel_diameter*1.25/4+wheel_diameter*0.125/2}" rpy="0 1.57 0 "/>
+            <origin xyz="0 0 ${-axle_offset}" rpy="0 1.57 0 "/>
         </joint>
         <link name="${name}_wheel">
@@ -145,4 +144,15 @@
         <!-- END RIGHT CAMERA -->
     </xacro:macro>
+    <!-- define suspension properties -->
+    <xacro:property name="wheel_diameter" value="0.33"/>
+    <xacro:property name="wheel_width" value="0.09"/>
+    <xacro:property name="yoke_height" value="0.3"/>
+    <xacro:property name="axle_offset" value="0.25"/>
+    <xacro:property name="suspension_length" value="0.35"/>
+    <xacro:property name="suspension_mounting_height" value="0.26"/>
+    <!-- instantiate 3 modules -->
+    <xacro:wheel_module name="stern" position="-1.3 0 ${suspension_mounting_height}"/>
+    <xacro:wheel_module name="port" position="0.0 0.5625 ${suspension_mounting_height}"/>
+    <xacro:wheel_module name="starboard" position="0.0 -0.5625 ${suspension_mounting_height}"/>
     <link name="base_link">
     </link>
@@ -150,5 +160,6 @@
         <parent link="base_link"/>
         <child link="body_triangle"/>
-        <origin xyz="1.5 0 0" rpy="0 0 0.0"/>
+        <origin xyz="0 0 ${wheel_diameter/2 + axle_offset + suspension_length - suspension_mounting_height}" rpy="0 0 0"/>
+        <!--<origin xyz="0 0 0" rpy="0 0 0"/>-->
     </joint>
     <!-- the big triangle -->
@@ -157,18 +168,23 @@
             <origin xyz="0.0 -0.75 0" rpy="0 0 1.57"/>
             <geometry>
-                <mesh filename="package://samplereturn/Media/models/triangle.mesh.xml" />
+                <mesh filename="package://samplereturn/Media/models/triangle.mesh.xml" scale="1 1 0.03"/>
             </geometry>
             <material name="plate"/>
         </visual>
     </link>
-    <!-- define suspension properties -->
-    <xacro:property name="wheel_diameter" value="0.33"/>
-    <xacro:property name="wheel_width" value="0.09"/>
-    <xacro:property name="yoke_thickness" value="0.1"/>
-    <xacro:property name="suspension_height" value="0.15"/>
-    <!-- instantiate 3 modules -->
-    <xacro:wheel_module name="stern" position="-1.3 0 0"/>
-    <xacro:wheel_module name="port" position="0.0 0.5625 0"/>
-    <xacro:wheel_module name="starboard" position="0.0 -0.5625 0"/>
+    <joint name="body_joint" type="fixed">
+        <parent link="body_triangle"/>
+        <child link="top_triangle"/>
+        <origin xyz="0 0 0.155" rpy="0 0 0"/>
+    </joint>
+    <link name="top_triangle">
+        <visual>
+            <origin xyz="0.0 -0.75 0" rpy="0 0 1.57"/>
+            <geometry>
+                <mesh filename="package://samplereturn/Media/models/triangle.mesh.xml" scale="1 1 0.03"/>
+            </geometry>
+            <material name="plate"/>
+        </visual>
+    </link>
     <!-- instantiate navigation pair -->
     <xacro:stereo_pair name="navigation" baseline="0.30" />

Commit message: Add gmapping

File: src/ros/samplereturn/urdf/robot.xacro (robot description, xacro)
@@ -245,4 +245,12 @@
         <origin xyz="0.10 0.0 1.0" rpy="-1.77 0 -1.57"/>
     </joint>
+    <!--fake laser scanner-->
+    <link name="fake_laser">
+    </link>
+    <joint name="fake_laser_joint" type="fixed">
+        <parent link="body_triangle"/>
+        <child link="fake_laser"/>
+        <origin xyz="0 0 0" rpy="-1.57 0 -1.57"/>
+    </joint>
     <!-- carousel -->
     <link name="carousel">

Commit message: Correct size of body triangles

File: src/ros/samplereturn/urdf/robot.xacro (robot description, xacro)
@@ -166,7 +166,7 @@
     <link name="body_triangle">
         <visual>
-            <origin xyz="0.0 -0.75 0" rpy="0 0 1.57"/>
-            <geometry>
-                <mesh filename="package://samplereturn/Media/models/triangle.mesh.xml" scale="1 1 0.03"/>
+            <origin xyz="0.0 -0.645 0" rpy="0 0 1.57"/>
+            <geometry>
+                <mesh filename="package://samplereturn/Media/models/triangle.mesh.xml" scale="0.86 0.75 0.03"/>
             </geometry>
             <material name="plate"/>
@@ -180,7 +180,7 @@
     <link name="top_triangle">
         <visual>
-            <origin xyz="0.0 -0.75 0" rpy="0 0 1.57"/>
-            <geometry>
-                <mesh filename="package://samplereturn/Media/models/triangle.mesh.xml" scale="1 1 0.03"/>
+            <origin xyz="0.0 -0.645 0" rpy="0 0 1.57"/>
+            <geometry>
+                <mesh filename="package://samplereturn/Media/models/triangle.mesh.xml" scale="0.86 0.75 0.03"/>
             </geometry>
             <material name="plate"/>
