Commit message: Tuning for visual odometry
Needs an orientation reference. visual odom cause the pose estimate to fly into
the air.

File: ros_workspace/src/samplereturn/urdf/robot.xacro (robot description, xacro)
@@ -155,4 +155,13 @@
     <xacro:wheel_module name="port" position="0.0 0.650 ${suspension_mounting_height}"/>
     <xacro:wheel_module name="starboard" position="0.0 -0.650 ${suspension_mounting_height}"/>
+    <!--
+    -->
+    <joint name="footprint_joint" type="fixed">
+        <parent link="base_footprint"/>
+        <child link="base_link"/>
+        <origin xyz="0 0 0" rpy="0 0 0"/>
+    </joint>
+    <link name="base_footprint">
+    </link>
     <link name="base_link">
     </link>
@@ -201,5 +210,5 @@
         -->
         <!-- so camera should be at 1.4 - deck -->
-        <origin xyz="0.015 0.0 0.990" rpy="-2.00 0 -1.57"/>
+        <origin xyz="0.015 0.0 0.990" rpy="-2.03 0 -1.57"/>
     </joint>
     <!-- instantiate manipulator pair -->

Commit message: Update for new manipulator camera mount

File: ros_workspace/src/samplereturn/urdf/robot.xacro (robot description, xacro)
@@ -204,5 +204,5 @@
     </joint>
     <!-- instantiate manipulator pair -->
-    <xacro:stereo_pair name="manipulator" baseline="0.30" />
+    <xacro:stereo_pair name="manipulator" baseline="0.05" />
     <!-- attach navigation pair -->
     <joint name="manipulator_stereo_pair_joint" type="fixed">
@@ -216,6 +216,5 @@
         suspension_height+wheel_diameter*1.25/2-wheel_diameter*0.125/2+wheel_diameter/2
         -->
-        <!-- so camera should be at 1.4 - deck -->
-        <origin xyz="-0.20 0.0 0.040" rpy="-2.80 0 -1.57"/>
+        <origin xyz="0.067 0.0 0.116" rpy="-2.80 0 -1.57"/>
     </joint>
     <link name="search_camera_body">

Commit message: DSLR pitched down an additional 10 degrees

File: ros_workspace/src/samplereturn/urdf/robot.xacro (robot description, xacro)
@@ -242,5 +242,5 @@
         <parent link="body_triangle"/>
         <child link="search_camera_body"/>
-        <origin xyz="0.10 0.0 1.0" rpy="-1.77 0 -1.57"/>
+        <origin xyz="0.10 0.0 1.0" rpy="-1.94 0 -1.57"/>
     </joint>
     <!--fake laser scanner-->

Commit message: Add coordinate frames for new cameras

File: ros_workspace/src/samplereturn/urdf/robot.xacro (robot description, xacro)
@@ -188,9 +188,11 @@
     </link>
     <!-- instantiate navigation pair -->
-    <xacro:stereo_pair name="navigation" baseline="0.30" />
+    <xacro:stereo_pair name="navigation_port" baseline="0.10" />
+    <xacro:stereo_pair name="navigation_bow" baseline="0.10" />
+    <xacro:stereo_pair name="navigation_starboard" baseline="0.10" />
     <!-- attach navigation pair -->
-    <joint name="navigation_stereo_pair_joint" type="fixed">
-        <parent link="body_triangle"/>
-        <child link="navigation_baseline_bar"/>
+    <joint name="navigation_port_stereo_pair_joint" type="fixed">
+        <parent link="body_triangle"/>
+        <child link="navigation_port_baseline_bar"/>
         <!-- macro defines camera with lenses facing along +z -->
         <!-- rpy is pi/2 + 16.5 degree down tilt -->
@@ -201,5 +203,31 @@
         -->
         <!-- so camera should be at 1.4 - deck -->
-        <origin xyz="0.015 0.0 0.990" rpy="-2.00 0 -1.57"/>
+        <origin xyz="0.125 0.160 0.810" rpy="-1.919 0 -0.522"/>
+    </joint>
+    <joint name="navigation_bow_stereo_pair_joint" type="fixed">
+        <parent link="body_triangle"/>
+        <child link="navigation_bow_baseline_bar"/>
+        <!-- macro defines camera with lenses facing along +z -->
+        <!-- rpy is pi/2 + 16.5 degree down tilt -->
+        <!-- height of bottom of deck (origin) is -->
+        <!-- suspension_height + yoke_height - yoke_offset + wheel_radius -->
+        <!--
+        suspension_height+wheel_diameter*1.25/2-wheel_diameter*0.125/2+wheel_diameter/2
+        -->
+        <!-- so camera should be at 1.4 - deck -->
+        <origin xyz="0.190 0.0 0.810" rpy="-1.919 0 -1.57"/>
+    </joint>
+    <joint name="navigation_starboard_stereo_pair_joint" type="fixed">
+        <parent link="body_triangle"/>
+        <child link="navigation_starboard_baseline_bar"/>
+        <!-- macro defines camera with lenses facing along +z -->
+        <!-- rpy is pi/2 + 16.5 degree down tilt -->
+        <!-- height of bottom of deck (origin) is -->
+        <!-- suspension_height + yoke_height - yoke_offset + wheel_radius -->
+        <!--
+        suspension_height+wheel_diameter*1.25/2-wheel_diameter*0.125/2+wheel_diameter/2
+        -->
+        <!-- so camera should be at 1.4 - deck -->
+        <origin xyz="0.125 -0.160 0.810" rpy="-1.919 0 -2.617"/>
     </joint>
     <!-- instantiate manipulator pair -->

Commit message: Change "bow" to "center"

File: ros_workspace/src/samplereturn/urdf/robot.xacro (robot description, xacro)
@@ -189,5 +189,5 @@
     <!-- instantiate navigation pair -->
     <xacro:stereo_pair name="navigation_port" baseline="0.10" />
-    <xacro:stereo_pair name="navigation_bow" baseline="0.10" />
+    <xacro:stereo_pair name="navigation_center" baseline="0.10" />
     <xacro:stereo_pair name="navigation_starboard" baseline="0.10" />
     <!-- attach navigation pair -->
@@ -205,7 +205,7 @@
         <origin xyz="0.125 0.160 0.810" rpy="-1.919 0 -0.522"/>
     </joint>
-    <joint name="navigation_bow_stereo_pair_joint" type="fixed">
-        <parent link="body_triangle"/>
-        <child link="navigation_bow_baseline_bar"/>
+    <joint name="navigation_center_stereo_pair_joint" type="fixed">
+        <parent link="body_triangle"/>
+        <child link="navigation_center_baseline_bar"/>
         <!-- macro defines camera with lenses facing along +z -->
         <!-- rpy is pi/2 + 16.5 degree down tilt -->

Commit message: Modified suspension properties to match Inventor model.

File: ros_workspace/src/samplereturn/urdf/robot.xacro (robot description, xacro)
@@ -145,10 +145,10 @@
     </xacro:macro>
     <!-- define suspension properties -->
-    <xacro:property name="wheel_diameter" value="0.33"/>
-    <xacro:property name="wheel_width" value="0.09"/>
+    <xacro:property name="wheel_diameter" value="0.3239"/>
+    <xacro:property name="wheel_width" value="0.12"/>
     <xacro:property name="yoke_height" value="0.3"/>
-    <xacro:property name="axle_offset" value="0.25"/>
-    <xacro:property name="suspension_length" value="0.35"/>
-    <xacro:property name="suspension_mounting_height" value="0.26"/>
+    <xacro:property name="axle_offset" value="0.255"/>
+    <xacro:property name="suspension_length" value="0.354"/>
+    <xacro:property name="suspension_mounting_height" value="0.276"/>
     <!-- instantiate 3 modules -->
     <xacro:wheel_module name="stern" position="-1.126 0 ${suspension_mounting_height}"/>

Commit message: Updated all camera positions to reflect Inventor model

File: ros_workspace/src/samplereturn/urdf/robot.xacro (robot description, xacro)
@@ -78,5 +78,5 @@
                 <geometry>
                     <!-- numbers measured from first prototype article -->
-                    <box size="${baseline-0.054} 0.0254 0.0381"/>
+                    <box size="${baseline+.076} 0.055 0.055"/>
                 </geometry>
                 <material name="sensor"/>
@@ -196,12 +196,9 @@
         <child link="navigation_port_baseline_bar"/>
         <!-- macro defines camera with lenses facing along +z -->
-        <!-- rpy is pi/2 + 16.5 degree down tilt -->
-        <!-- height of bottom of deck (origin) is -->
-        <!-- suspension_height + yoke_height - yoke_offset + wheel_radius -->
-        <!--
-        suspension_height+wheel_diameter*1.25/2-wheel_diameter*0.125/2+wheel_diameter/2
-        -->
-        <!-- so camera should be at 1.4 - deck -->
-        <origin xyz="0.125 0.160 0.810" rpy="-1.919 0 -0.522"/>
+        <!-- rpy is pi/2 + T degrees down tilt -->
+        <!-- year 3 triple nav setup is tilted down 20 degrees -->
+        <!-- in plane of camera centers, baselines point 60 deg apart -->
+        <!-- all nav cameras are 1.303m off dirt by Inventor model (no settling)-->
+        <origin xyz="0.0956 0.1553 0.8085" rpy="-1.919 0 -0.523"/>
     </joint>
     <joint name="navigation_center_stereo_pair_joint" type="fixed">
@@ -209,12 +206,9 @@
         <child link="navigation_center_baseline_bar"/>
         <!-- macro defines camera with lenses facing along +z -->
-        <!-- rpy is pi/2 + 16.5 degree down tilt -->
-        <!-- height of bottom of deck (origin) is -->
-        <!-- suspension_height + yoke_height - yoke_offset + wheel_radius -->
-        <!--
-        suspension_height+wheel_diameter*1.25/2-wheel_diameter*0.125/2+wheel_diameter/2
-        -->
-        <!-- so camera should be at 1.4 - deck -->
-        <origin xyz="0.190 0.0 0.810" rpy="-1.919 0 -1.57"/>
+        <!-- rpy is pi/2 + T degrees down tilt -->
+        <!-- year 3 triple nav setup is tilted down 20 degrees -->
+        <!-- in plane of camera centers, baselines point 60 deg apart -->
+        <!-- all nav cameras are 1.303m off dirt by Inventor model (no settling)-->
+        <origin xyz="0.1788 0.0 0.8085" rpy="-1.919 0 -1.57"/>
     </joint>
     <joint name="navigation_starboard_stereo_pair_joint" type="fixed">
@@ -222,12 +216,9 @@
         <child link="navigation_starboard_baseline_bar"/>
         <!-- macro defines camera with lenses facing along +z -->
-        <!-- rpy is pi/2 + 16.5 degree down tilt -->
-        <!-- height of bottom of deck (origin) is -->
-        <!-- suspension_height + yoke_height - yoke_offset + wheel_radius -->
-        <!--
-        suspension_height+wheel_diameter*1.25/2-wheel_diameter*0.125/2+wheel_diameter/2
-        -->
-        <!-- so camera should be at 1.4 - deck -->
-        <origin xyz="0.125 -0.160 0.810" rpy="-1.919 0 -2.617"/>
+        <!-- rpy is pi/2 + T degrees down tilt -->
+        <!-- year 3 triple nav setup is tilted down 20 degrees -->
+        <!-- in plane of camera centers, baselines point 60 deg apart -->
+        <!-- all nav cameras are 1.303m off dirt by Inventor model (no settling)-->
+         <origin xyz="0.0956 -0.1553 0.8085" rpy="-1.919 0 -2.618"/>
     </joint>
     <!-- instantiate manipulator pair -->
@@ -238,11 +229,8 @@
         <child link="manipulator_baseline_bar"/>
         <!-- macro defines camera with lenses facing along +z -->
-        <!-- rpy is pi/2 + 16.5 degree down tilt -->
-        <!-- height of bottom of deck (origin) is -->
-        <!-- suspension_height + yoke_height - yoke_offset + wheel_radius -->
-        <!--
-        suspension_height+wheel_diameter*1.25/2-wheel_diameter*0.125/2+wheel_diameter/2
-        -->
-        <origin xyz="0.067 0.0 0.116" rpy="-2.80 0 -1.57"/>
+        <!-- rpy is pi/2 + T degrees down tilt -->
+        <!-- note: year 3 manipulator is tilted down 70 degrees -->
+        <!-- manipulators are .555m off dirt by Inventor model (no settling)-->
+        <origin xyz="-0.1147 0.0 0.0605" rpy="-2.79 0 -1.57"/>
     </joint>
     <link name="search_camera_body">
@@ -270,5 +258,6 @@
         <parent link="body_triangle"/>
         <child link="search_camera_body"/>
-        <origin xyz="0.10 0.0 1.0" rpy="-1.94 0 -1.57"/>
+        <!-- still considering 3 search camera angles: 20, 25, 40 degrees -->
+        <origin xyz="0.1763 0.0 0.9203" rpy="-2.01 0 -1.57"/>
     </joint>
     <!--fake laser scanner-->

Commit message: The search camera angle is 20 degrees, not 25 below horizon

File: ros_workspace/src/samplereturn/urdf/robot.xacro (robot description, xacro)
@@ -259,5 +259,5 @@
         <child link="search_camera_body"/>
         <!-- still considering 3 search camera angles: 20, 25, 40 degrees -->
-        <origin xyz="0.1763 0.0 0.9203" rpy="-2.01 0 -1.57"/>
+        <origin xyz="0.1763 0.0 0.9203" rpy="-1.92 0 -1.57"/>
     </joint>
     <!--fake laser scanner-->

Commit message: Corrected manipulator offset

File: ros_workspace/src/samplereturn/urdf/robot.xacro (robot description, xacro)
@@ -180,9 +180,23 @@
     <link name="top_triangle">
         <visual>
-            <origin xyz="0.0 -0.645 0" rpy="0 0 1.57"/>
+            <origin xyz="0 -0.645 0" rpy="0 0 1.57"/>
             <geometry>
                 <mesh filename="package://samplereturn/Media/models/triangle.mesh.xml" scale="0.86 0.75 0.03"/>
             </geometry>
             <material name="plate"/>
+        </visual>
+    </link>
+    <joint name="manipulator_joint" type="fixed">
+        <parent link="body_triangle"/>
+        <child link="manipulator_arm"/>
+        <origin xyz="0.06666666 0 0" rpy="0 0 0"/>
+    </joint>
+    <link name="manipulator_arm">
+        <visual>
+            <origin xyz="0 0 0" rpy="0 0 1.57"/>
+            <geometry>
+                <mesh filename="package://samplereturn/Media/models/triangle.mesh.xml" scale="0.05 0.05 10"/>
+            </geometry>
+            <material name="suspension"/>
         </visual>
     </link>

Commit message: Manipulator camera position re-measurement

File: ros_workspace/src/samplereturn/urdf/robot.xacro (robot description, xacro)
@@ -163,5 +163,5 @@
         <!--<origin xyz="0 0 0" rpy="0 0 0"/>-->
     </joint>
-    <!-- the big triangle -->
+    <!-- bottom plate of robot, upper surface -->
     <link name="body_triangle">
         <visual>
@@ -246,5 +246,5 @@
         <!-- note: year 3 manipulator is tilted down 70 degrees -->
         <!-- manipulators are .555m off dirt by Inventor model (no settling)-->
-        <origin xyz="-0.1147 0.0 0.0605" rpy="-2.79 0 -1.57"/>
+        <origin xyz="-0.1147 0.0 0.064" rpy="-2.792 0 -1.571"/>
     </joint>
     <link name="search_camera_body">

Commit message: Corrected search_camera urdf

File: ros_workspace/src/samplereturn/urdf/robot.xacro (robot description, xacro)
@@ -248,5 +248,5 @@
         <origin xyz="-0.1147 0.0 0.064" rpy="-2.792 0 -1.571"/>
     </joint>
-    <link name="search_camera_body">
+    <link name="search_camera">
         <visual>
             <geometry>
@@ -265,5 +265,5 @@
     </link>
     <joint name="search_lens_joint" type="fixed">
-        <parent link="search_camera_body"/>
+        <parent link="search_camera"/>
         <child link="search_camera_lens"/>
         <origin xyz="0.0 0.0 0.025" rpy="0 0 0"/>
@@ -271,7 +271,7 @@
     <joint name="search_camera_joint" type="fixed">
         <parent link="body_triangle"/>
-        <child link="search_camera_body"/>
+        <child link="search_camera"/>
         <!-- still considering 3 search camera angles: 20, 25, 40 degrees -->
-        <origin xyz="0.1763 0.0 0.9203" rpy="-1.92 0 -1.57"/>
+        <origin xyz="0.124 0.0 0.963" rpy="-1.92 0 -1.571"/>
     </joint>
     <!--fake laser scanner-->

Commit message: Adjust search camera yaw

File: ros_workspace/src/samplereturn/urdf/robot.xacro (robot description, xacro)
@@ -273,5 +273,5 @@
         <child link="search_camera"/>
         <!-- still considering 3 search camera angles: 20, 25, 40 degrees -->
-        <origin xyz="0.124 0.0 0.963" rpy="-1.92 0 -1.571"/>
+        <origin xyz="0.124 0.0 0.963" rpy="-1.92 0 -1.515"/>
     </joint>
     <!--fake laser scanner-->

Commit message: Way too many 6s in manip. offset, possibly satanic
Actually, I'm bad at vim.

File: ros_workspace/src/samplereturn/urdf/robot.xacro (robot description, xacro)
@@ -190,5 +190,5 @@
         <parent link="body_triangle"/>
         <child link="manipulator_arm"/>
-        <origin xyz="0.06666666 0 0" rpy="0 0 0"/>
+        <origin xyz="0.066 0 0" rpy="0 0 0"/>
     </joint>
     <link name="manipulator_arm">

Commit message: Adjust body_triangle elevation

File: ros_workspace/src/samplereturn/urdf/robot.xacro (robot description, xacro)
@@ -148,7 +148,7 @@
     <xacro:property name="wheel_width" value="0.12"/>
     <xacro:property name="yoke_height" value="0.3"/>
-    <xacro:property name="axle_offset" value="0.255"/>
-    <xacro:property name="suspension_length" value="0.354"/>
-    <xacro:property name="suspension_mounting_height" value="0.276"/>
+    <xacro:property name="axle_offset" value="0.254"/>
+    <xacro:property name="suspension_length" value="0.318"/>
+    <xacro:property name="suspension_mounting_height" value="0.256"/>
     <!-- instantiate 3 modules -->
     <xacro:wheel_module name="stern" position="-1.126 0 ${suspension_mounting_height}"/>

Commit message: Adjust search camera pointing
Used 8m distance measured with SimpleMove server.

Also add useful launch to update tf on running robot.

File: ros_workspace/src/samplereturn/urdf/robot.xacro (robot description, xacro)
@@ -273,5 +273,5 @@
         <child link="search_camera"/>
         <!-- still considering 3 search camera angles: 20, 25, 40 degrees -->
-        <origin xyz="0.124 0.0 0.963" rpy="-1.92 0 -1.515"/>
+        <origin xyz="0.124 0.0 0.963" rpy="-1.9185 0 -1.634"/>
     </joint>
     <!--fake laser scanner-->

Commit message: Add imu mounting points to URDF

File: ros_workspace/src/samplereturn/urdf/robot.xacro (robot description, xacro)
@@ -298,3 +298,15 @@
         <origin xyz="-0.239 0.0 -0.121"/>
     </joint>
+    <link name="imu_0"/>
+    <joint name="imu_0_mount" type="fixed">
+        <parent link="body_triangle"/>
+        <child link="imu_0"/>
+        <origin xyz="-0.445 0 0.0113" rpy="0 3.1416 -1.5708"/>
+    </joint>
+    <link name="imu_1"/>
+    <joint name="imu_1_mount" type="fixed">
+        <parent link="body_triangle"/>
+        <child link="imu_1"/>
+        <origin xyz="-0.445 0 0.0175" rpy="0 3.1416 -1.5708"/>
+    </joint>
 </robot>

Commit message: Add microstrain frame to urdf

File: ros_workspace/src/samplereturn/urdf/robot.xacro (robot description, xacro)
@@ -310,3 +310,9 @@
         <origin xyz="-0.445 0 0.0175" rpy="0 3.1416 -1.5708"/>
     </joint>
+    <link name="microstrain"/>
+    <joint name="microstrain_mount" type="fixed">
+        <parent link="body_triangle"/>
+        <child link="microstrain"/>
+        <origin xyz="-0.455 0 0.155" rpy="0 3.1416 0"/>
+    </joint>
 </robot>

Commit message: Add microstrain frame to urdf
and add frame id to launch

File: ros_workspace/src/samplereturn/urdf/robot.xacro (robot description, xacro)
@@ -300,3 +300,9 @@
         <origin xyz="-0.445 0 0.0175" rpy="0 3.1416 -1.5708"/>
     </joint>
+    <link name="microstrain"/>
+    <joint name="microstrain_mount" type="fixed">
+        <parent link="body_triangle"/>
+        <child link="microstrain"/>
+        <origin xyz="-0.455 0 0.155" rpy="0 3.1416 0"/>
+    </joint>
 </robot>

Commit message: New nav camera mount URDF

File: ros_workspace/src/samplereturn/urdf/robot.xacro (robot description, xacro)
@@ -205,34 +205,24 @@
     <xacro:stereo_pair name="navigation_center" baseline="0.10" />
     <xacro:stereo_pair name="navigation_starboard" baseline="0.10" />
-    <!-- attach navigation pair -->
+    <!-- attach navigation pairs as follows: -->
+    <!-- macro defines camera with lenses facing along +z -->
+    <!-- rpy is pi/2 + T degrees down tilt -->
+    <!-- year 4 triple nav setup is tilted down 20 degrees -->
+    <!-- in plane of camera centers, side baselines point 47 deg out -->
+    <!-- all nav cameras are .861m off of the lower frame plate-->
     <joint name="navigation_port_stereo_pair_joint" type="fixed">
         <parent link="body_triangle"/>
         <child link="navigation_port_baseline_bar"/>
-        <!-- macro defines camera with lenses facing along +z -->
-        <!-- rpy is pi/2 + T degrees down tilt -->
-        <!-- year 3 triple nav setup is tilted down 20 degrees -->
-        <!-- in plane of camera centers, baselines point 60 deg apart -->
-        <!-- all nav cameras are 1.303m off dirt by Inventor model (no settling)-->
-        <origin xyz="0.0956 0.1553 0.8085" rpy="-1.919 0 -0.523"/>
+        <origin xyz="0.0761 0.1568 0.8608" rpy="-1.919 0 -0.7505"/>
     </joint>
     <joint name="navigation_center_stereo_pair_joint" type="fixed">
         <parent link="body_triangle"/>
         <child link="navigation_center_baseline_bar"/>
-        <!-- macro defines camera with lenses facing along +z -->
-        <!-- rpy is pi/2 + T degrees down tilt -->
-        <!-- year 3 triple nav setup is tilted down 20 degrees -->
-        <!-- in plane of camera centers, baselines point 60 deg apart -->
-        <!-- all nav cameras are 1.303m off dirt by Inventor model (no settling)-->
-        <origin xyz="0.1788 0.0 0.8085" rpy="-1.919 0 -1.57"/>
+        <origin xyz="0.141 0.0 0.8608" rpy="-1.919 0 -1.5708"/>
     </joint>
     <joint name="navigation_starboard_stereo_pair_joint" type="fixed">
         <parent link="body_triangle"/>
         <child link="navigation_starboard_baseline_bar"/>
-        <!-- macro defines camera with lenses facing along +z -->
-        <!-- rpy is pi/2 + T degrees down tilt -->
-        <!-- year 3 triple nav setup is tilted down 20 degrees -->
-        <!-- in plane of camera centers, baselines point 60 deg apart -->
-        <!-- all nav cameras are 1.303m off dirt by Inventor model (no settling)-->
-         <origin xyz="0.0956 -0.1553 0.8085" rpy="-1.919 0 -2.618"/>
+         <origin xyz="0.0761 -0.1568 0.8608" rpy="-1.919 0 -2.3911"/>
     </joint>
     <!-- instantiate manipulator pair -->

Commit message: URDF change for new wheel yokes

File: ros_workspace/src/samplereturn/urdf/robot.xacro (robot description, xacro)
@@ -147,5 +147,5 @@
     <xacro:property name="wheel_diameter" value="0.3239"/>
     <xacro:property name="wheel_width" value="0.12"/>
-    <xacro:property name="yoke_height" value="0.3"/>
+    <xacro:property name="yoke_height" value="0.281"/>
     <xacro:property name="axle_offset" value="0.254"/>
     <xacro:property name="suspension_length" value="0.318"/>

Commit message: Initial link for sun camera

File: ros_workspace/src/samplereturn/urdf/robot.xacro (robot description, xacro)
@@ -305,4 +305,10 @@
         <child link="microstrain"/>
         <origin xyz="-0.455 0 0.155" rpy="0 3.1416 0"/>
-    </joint>
+     </joint>
+     <link name="sun_camera"/>
+     <joint name="sun_camera_bracket" type="fixed">
+         <parent link="body_triangle"/>
+         <child link="sun_camera"/>
+         <origin xyz="-0.727 0 0.311" rpy="0 0 1.57"/>
+     </joint>
 </robot>

Commit message: Removed unused IMU urdf entries

File: ros_workspace/src/samplereturn/urdf/robot.xacro (robot description, xacro)
@@ -288,16 +288,4 @@
         <origin xyz="-0.239 0.0 -0.121"/>
     </joint>
-    <link name="imu_0"/>
-    <joint name="imu_0_mount" type="fixed">
-        <parent link="body_triangle"/>
-        <child link="imu_0"/>
-        <origin xyz="-0.445 0 0.0113" rpy="0 3.1416 -1.5708"/>
-    </joint>
-    <link name="imu_1"/>
-    <joint name="imu_1_mount" type="fixed">
-        <parent link="body_triangle"/>
-        <child link="imu_1"/>
-        <origin xyz="-0.445 0 0.0175" rpy="0 3.1416 -1.5708"/>
-    </joint>
     <link name="microstrain"/>
     <joint name="microstrain_mount" type="fixed">
