Commit message: Reset search camera URDF to default

File: ros_workspace/src/samplereturn/urdf/robot.xacro (robot description, xacro)
@@ -263,6 +263,6 @@
         <parent link="body_triangle"/>
         <child link="search_camera"/>
-        <!-- still considering 3 search camera angles: 20, 25, 40 degrees -->
-        <origin xyz="0.124 0.0 0.963" rpy="-1.9185 0 -1.634"/>
+        <!--  search camera angles:  20 degrees -->
+        <origin xyz="0.124 0.0 0.963" rpy="-1.920 0 -1.5708"/>
     </joint>
     <!--fake laser scanner-->

Commit message: New URDF data for triple search camera array

File: ros_workspace/src/samplereturn/urdf/robot.xacro (robot description, xacro)
@@ -239,30 +239,88 @@
         <origin xyz="-0.1147 0.0 0.064" rpy="-2.792 0 -1.571"/>
     </joint>
-    <link name="search_camera">
-        <visual>
-            <geometry>
-                <box size="0.10 0.08 0.05"/>
+    <!-- begin seach and beacon cameras -->
+    <!-- center camera -->
+    <link name="search_center_camera">
+        <visual>
+            <geometry>
+                <box size="0.03 0.03 0.03"/>
             </geometry>
             <material name="sensor"/>
         </visual>
     </link>
-    <link name="search_camera_lens">
-        <visual>
-            <geometry>
-                <cylinder length="0.10" radius="0.035"/>
+    <link name="search_center_lens">
+        <visual>
+            <geometry>
+                <cylinder length="0.04" radius="0.015"/>
             </geometry>
             <material name="lens"/>
         </visual>
     </link>
-    <joint name="search_lens_joint" type="fixed">
-        <parent link="search_camera"/>
-        <child link="search_camera_lens"/>
-        <origin xyz="0.0 0.0 0.025" rpy="0 0 0"/>
-    </joint>
-    <joint name="search_camera_joint" type="fixed">
-        <parent link="body_triangle"/>
-        <child link="search_camera"/>
-        <!--  search camera angles:  20 degrees -->
-        <origin xyz="0.124 0.0 0.963" rpy="-1.920 0 -1.5708"/>
+    <joint name="search_center_lens_joint" type="fixed">
+        <parent link="search_center_camera"/>
+        <child link="search_center_lens"/>
+        <origin xyz="0.0 0.0 0.04" rpy="0 0 0"/>
+    </joint>
+    <joint name="search_center_camera_joint" type="fixed">
+        <parent link="body_triangle"/>
+        <child link="search_center_camera"/>
+        <!--  search camera center angle:  45 degrees -->
+        <origin xyz="0.207 0.0 0.970" rpy="-2.3562 0 -1.5708"/>
+    </joint>
+    <!-- port camera -->
+    <link name="search_port_camera">
+        <visual>
+            <geometry>
+                <box size="0.03 0.03 0.03"/>
+            </geometry>
+            <material name="sensor"/>
+        </visual>
+    </link>
+    <link name="search_port_lens">
+        <visual>
+            <geometry>
+                <cylinder length="0.04" radius="0.015"/>
+            </geometry>
+            <material name="lens"/>
+        </visual>
+    </link>
+    <joint name="search_port_lens_joint" type="fixed">
+        <parent link="search_port_camera"/>
+        <child link="search_port_lens"/>
+        <origin xyz="0.0 0.0 0.04" rpy="0 0 0"/>
+    </joint>
+    <joint name="search_port_camera_joint" type="fixed">
+        <parent link="body_triangle"/>
+        <child link="search_port_camera"/>
+        <!--  search camera center angle:  45 degrees -->
+        <origin xyz="0.178 0.070 0.971" rpy="-2.2689 0 -0.5236"/>
+    </joint>
+    <!-- starboard camera -->
+    <link name="search_starboard_camera">
+        <visual>
+            <geometry>
+                <box size="0.03 0.03 0.03"/>
+            </geometry>
+            <material name="sensor"/>
+        </visual>
+    </link>
+    <link name="search_starboard_lens">
+        <visual>
+            <geometry>
+                <cylinder length="0.04" radius="0.015"/>
+            </geometry>
+            <material name="lens"/>
+        </visual>
+    </link>
+    <joint name="search_starboard_lens_joint" type="fixed">
+        <parent link="search_starboard_camera"/>
+        <child link="search_starboard_lens"/>
+        <origin xyz="0.0 0.0 0.04" rpy="0 0 0"/>
+    </joint>
+    <joint name="search_starboard_camera_joint" type="fixed">
+        <parent link="body_triangle"/>
+        <child link="search_starboard_camera"/>
+        <!--  search camera center angle:  45 degrees -->
+        <origin xyz="0.178 -0.070 0.971" rpy="-2.2689 0 -2.6180"/>
     </joint>
     <!--fake laser scanner-->

Commit message: Added beacon camera: navigation_beacon_camera

File: ros_workspace/src/samplereturn/urdf/robot.xacro (robot description, xacro)
@@ -293,5 +293,5 @@
         <parent link="body_triangle"/>
         <child link="search_port_camera"/>
-        <!--  search camera center angle:  45 degrees -->
+        <!--  search camera side angles:  40 deg. down, 60 deg. out -->
         <origin xyz="0.178 0.070 0.971" rpy="-2.2689 0 -0.5236"/>
     </joint>
@@ -321,6 +321,34 @@
         <parent link="body_triangle"/>
         <child link="search_starboard_camera"/>
-        <!--  search camera center angle:  45 degrees -->
+        <!--  search camera side angles:  40 deg. down, 60 deg. out -->
         <origin xyz="0.178 -0.070 0.971" rpy="-2.2689 0 -2.6180"/>
+    </joint>
+    <!-- beacon camera -->
+    <link name="navigation_beacon_camera">
+        <visual>
+            <geometry>
+                <box size="0.03 0.03 0.03"/>
+            </geometry>
+            <material name="sensor"/>
+        </visual>
+    </link>
+    <link name="navigation_beacon_lens">
+        <visual>
+            <geometry>
+                <cylinder length="0.04" radius="0.015"/>
+            </geometry>
+            <material name="lens"/>
+        </visual>
+    </link>
+    <joint name="navigation_beacon_lens_joint" type="fixed">
+        <parent link="navigation_beacon_camera"/>
+        <child link="navigation_beacon_lens"/>
+        <origin xyz="0.0 0.0 0.04" rpy="0 0 0"/>
+    </joint>
+    <joint name="navigation_beacon_camera_joint" type="fixed">
+        <parent link="body_triangle"/>
+        <child link="navigation_beacon_camera"/>
+        <!--  navigation beacon angle:  0 degrees -->
+        <origin xyz="0.165 0 0.899" rpy="-1.5708 -0 -1.5708"/>
     </joint>
     <!--fake laser scanner-->

Commit message: Add phidget to URDF

File: ros_workspace/src/samplereturn/urdf/robot.xacro (robot description, xacro)
@@ -381,4 +381,10 @@
         <origin xyz="-0.455 0 0.155" rpy="0 3.1416 0"/>
      </joint>
+    <link name="imu_0"/>
+    <joint name="imu_0_mount" type="fixed">
+        <parent link="body_triangle"/>
+        <child link="imu_0"/>
+        <origin xyz="-0.445 0 0.0113" rpy="0 3.1416 -1.5708"/>
+    </joint>
      <link name="sun_camera"/>
      <joint name="sun_camera_bracket" type="fixed">

Commit message: Fix IMU mounting transform

File: ros_workspace/src/samplereturn/urdf/robot.xacro (robot description, xacro)
@@ -385,5 +385,5 @@
         <parent link="body_triangle"/>
         <child link="imu_0"/>
-        <origin xyz="-0.445 0 0.0113" rpy="0 3.1416 -1.5708"/>
+        <origin xyz="-0.445 0 0.0113" rpy="3.1416 0 -1.5708"/>
     </joint>
      <link name="sun_camera"/>

Commit message: Correct mounting of gyro and invert imu

File: ros_workspace/src/samplereturn/urdf/robot.xacro (robot description, xacro)
@@ -385,5 +385,11 @@
         <parent link="body_triangle"/>
         <child link="imu_0"/>
-        <origin xyz="-0.445 0 0.0113" rpy="3.1416 0 -1.5708"/>
+        <origin xyz="-0.445 0 0.0113" rpy="0 0 1.5708"/>
+    </joint>
+    <link name="gyro"/>
+    <joint name="gyro_mount" type="fixed">
+        <parent link="body_triangle"/>
+        <child link="gyro"/>
+        <origin xyz="-.635 0.127 0" rpy="3.1416 0 0"/>
     </joint>
      <link name="sun_camera"/>
