Commit message: Bolt beacon down to map

File: ros_workspace/src/samplereturn/urdf/beacon.urdf (robot description, URDF)
Before this commit: robot home_beacon, 3 links, 2 joints
Links:
- added link map
Joints:
- added joint beacon_bolts: type fixed, parent map, child beacon, origin xyz=0.0 0.0 0.0 rpy=0.0 0.0 0.0

Commit message: Added all beacon tags

File: ros_workspace/src/samplereturn/urdf/beacon.urdf (robot description, URDF)
Before this commit: robot home_beacon, 4 links, 3 joints
Links:
- added link beacon_back
- added link beacon_front_left
- added link beacon_left
- added link beacon_right
Joints:
- removed joint beacon_bolts
- added joint beacon_back: type fixed, parent beacon, child beacon_back, origin xyz=0.0 0.0 0.394 rpy=0.0 3.1416 0.0
- added joint beacon_front_left: type fixed, parent beacon, child beacon_front_left, origin xyz=0.610 0.0 0.0 rpy=0.0 0.0 0.0
- added joint beacon_left: type fixed, parent beacon, child beacon_left, origin xyz=0.775 0.0 0.197 rpy=0.0 -1.5708 0.0
- added joint beacon_mount: type fixed, parent map, child beacon, origin xyz=-1.30 0.0 1.243 rpy=-1.5708 0 1.5708
- added joint beacon_right: type fixed, parent beacon, child beacon_right, origin xyz=-0.775 0.0 0.197 rpy=0.0 1.5708 0.0
- joint beacon_front_right_x: origin xyz=0.6096 0.0 0.0 rpy=0.0 0.0 0.0 -> xyz=-0.610 0.0 0.0 rpy=0.0 0.0 0.0

Commit message: New beacon frames

File: ros_workspace/src/samplereturn/urdf/beacon.urdf (robot description, URDF)
Before this commit: robot home_beacon, 8 links, 7 joints
Links:
- removed link beacon_back
- removed link beacon_front
- removed link beacon_left
- removed link beacon_right
- added link beacon_back_left
- added link beacon_back_right
- added link beacon_left_bottom
- added link beacon_left_top
- added link beacon_right_bottom
- added link beacon_right_top
Joints:
- removed joint beacon_back
- removed joint beacon_front_left
- removed joint beacon_front_x
- removed joint beacon_left
- removed joint beacon_right
- added joint beacon_back_left_x: type fixed, parent beacon, child beacon_back_left, origin xyz=0.0 -0.366 0.394 rpy=0.0 3.1416 0.0
- added joint beacon_back_right_x: type fixed, parent beacon, child beacon_back_right, origin xyz=0.0 0.366 0.394 rpy=0.0 3.1416 0.0
- added joint beacon_front_left_x: type fixed, parent beacon, child beacon_front_left, origin xyz=0.366 0.0 0.0 rpy=0.0 0.0 0.0
- added joint beacon_left_bottom_x: type fixed, parent beacon, child beacon_left_bottom, origin xyz=0.775 -0.229 0.197 rpy=0.0 -1.5708 0.0
- added joint beacon_left_top_x: type fixed, parent beacon, child beacon_left_top, origin xyz=0.775 0.229 0.197 rpy=0.0 -1.5708 0.0
- added joint beacon_right_bottom: type fixed, parent beacon, child beacon_right_bottom, origin xyz=-0.775 -0.229 0.197 rpy=0.0 1.5708 0.0
- added joint beacon_right_top_x: type fixed, parent beacon, child beacon_right_top, origin xyz=-0.775 0.229 0.197 rpy=0.0 1.5708 0.0
- joint beacon_front_right_x: origin xyz=-0.610 0.0 0.0 rpy=0.0 0.0 0.0 -> xyz=-0.366 0.0 0.0 rpy=0.0 0.0 0.0

Commit message: Corrected beacon poses

File: ros_workspace/src/samplereturn/urdf/beacon.urdf (robot description, URDF)
Before this commit: robot home_beacon, 10 links, 9 joints
Joints:
- joint beacon_back_left_x: origin xyz=0.0 -0.366 0.394 rpy=0.0 3.1416 0.0 -> xyz=0.366 0.0 0.394 rpy=0.0 3.1416 0.0
- joint beacon_back_right_x: origin xyz=0.0 0.366 0.394 rpy=0.0 3.1416 0.0 -> xyz=-0.366 0.0 0.394 rpy=0.0 3.1416 0.0
- joint beacon_left_bottom_x: origin xyz=0.775 -0.229 0.197 rpy=0.0 -1.5708 0.0 -> xyz=0.775 0.229 0.197 rpy=0.0 -1.5708 0.0
- joint beacon_left_top_x: origin xyz=0.775 0.229 0.197 rpy=0.0 -1.5708 0.0 -> xyz=0.775 -0.229 0.197 rpy=0.0 -1.5708 0.0
- joint beacon_right_bottom: origin xyz=-0.775 -0.229 0.197 rpy=0.0 1.5708 0.0 -> xyz=-0.775 0.229 0.197 rpy=0.0 1.5708 0.0
- joint beacon_right_top_x: origin xyz=-0.775 0.229 0.197 rpy=0.0 1.5708 0.0 -> xyz=-0.775 -0.229 0.197 rpy=0.0 1.5708 0.0

Commit message: New tags, under beacon, slanted

File: ros_workspace/src/samplereturn/urdf/beacon.urdf (robot description, URDF)
Before this commit: robot home_beacon, 10 links, 9 joints
Links:
- added link beacon_back_lower
- added link beacon_front_lower
Joints:
- added joint beacon_back_lower_x: type fixed, parent beacon, child beacon_back_lower, origin xyz=0.0 0.803 0.197 rpy=0.0 2.8784 0.0
- added joint beacon_front_lower_x: type fixed, parent beacon, child beacon_front_lower, origin xyz=0.0 0.803 0.197 rpy=0.0 -0.2632 0.0

Commit message: Insert transform from platform to map

File: ros_workspace/src/samplereturn/urdf/beacon.urdf (robot description, URDF)
Before this commit: robot home_beacon, 12 links, 11 joints
Links:
- removed link map
- added link platform
Joints:
- joint beacon_mount: parent map -> platform

File: ros_workspace/src/samplereturn/urdf/sim_beacon.urdf (robot description, URDF)
Before this commit: robot home_beacon, 12 links, 11 joints
Links:
- removed link sim_map
- added link platform
Joints:
- joint beacon_mount: parent sim_map -> platform

Commit message: New hex beacon description

File: ros_workspace/src/samplereturn/urdf/beacon.urdf (robot description, URDF)
Before this commit: robot home_beacon, 12 links, 11 joints
Links:
- removed link beacon_back_lower
- removed link beacon_front_lower
- removed link beacon_left_bottom
- removed link beacon_left_top
- removed link beacon_right_bottom
- removed link beacon_right_top
- added link beacon_back
- added link beacon_front
Joints:
- removed joint beacon_back_lower_x
- removed joint beacon_front_lower_x
- removed joint beacon_left_bottom_x
- removed joint beacon_left_top_x
- removed joint beacon_right_bottom
- removed joint beacon_right_top_x
- added joint beacon_back_x: type fixed, parent beacon, child beacon_back, origin xyz=0.0 0.0 0.404 rpy=0.0 3.1416 0.0
- added joint beacon_front_x: type fixed, parent beacon, child beacon_front, origin xyz=0.0 0.0 0.0 rpy=0.0 0.0 0.0
- joint beacon_back_left_x: origin xyz=0.366 0.0 0.394 rpy=0.0 3.1416 0.0 -> xyz=0.652 0.0 0.305 rpy=0.0 -2.8381 0.0
- joint beacon_back_right_x: origin xyz=-0.366 0.0 0.394 rpy=0.0 3.1416 0.0 -> xyz=-0.652 0.0 0.305 rpy=0.0 2.8381 0.0
- joint beacon_front_left_x: origin xyz=0.366 0.0 0.0 rpy=0.0 0.0 0.0 -> xyz=0.652 0.0 0.100 rpy=0.0 -0.3035 0.0
- joint beacon_front_right_x: origin xyz=-0.366 0.0 0.0 rpy=0.0 0.0 0.0 -> xyz=-0.652 0.0 .100 rpy=0.0 0.3035 0.0
- joint beacon_mount: origin xyz=-1.30 0.0 1.243 rpy=-1.5708 0 1.5708 -> xyz=-1.30 0.0 0.942 rpy=-1.5708 0 1.5708
